File: kicad/usb-led-controller.kicad_pcb (KiCad board)
At the start: 4 copper layers, 70 x 30 mm, 109 parts, among them J1 SWD, J2 PWR, J3 USB, J4 PWM_0, J5 PWM_1, J6 WS2812_0, J7 WS2812_1, Q1 NVS4409N, Q2 NVS4409N, Q3 NVS4409N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

Commit message: Added some pullups
Parts:
- added R12: 10K, Resistor_SMD:R_0402_1005Metric, F.Cu at (164.5, 117.3)
- added R13: 10K, Resistor_SMD:R_0402_1005Metric, F.Cu at (164.5, 120.1)
- added REF**: VIA-0.3_0.6-TENT, usb-led-controller:VIA-0.3_0.6-TENT, F.Cu at (165.0, 119.2)
- added REF**: VIA-0.3_0.6-TENT, usb-led-controller:VIA-0.3_0.6-TENT, F.Cu at (165.0, 116.4)
Routing:
- net /WS2812_DATA_INV: track 13.6 -> 16.4 mm
- net +3V3: track 2.06 -> 3.86 mm
- net /WS2812_0_~OE: track 28.5 -> 30.0 mm
- net /WS2812_1_~OE: track 18.6 -> 19.8 mm

Commit message: Adding text to silkscreen
Other:
- board text added: "12V GND GND GND"
- board text added: "12V PWM 0"
- board text added: "12V PWM 1"
- board text added: "5V D- D+ GND"
- board text added: "B R G 12V"
- board text added: "GND DATA 5V"
- board text added: "LED Power"
- board text added: "Rev A"
- board text added: "USB"
- board text added: "USB LED Controller"
- board text added: "WS2812 0"
- board text added: "WS2812 1"
- board text added: "http://kevincuzner.com"
Changed lines of the file:
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@@
-(kicad_pcb (version 20171130) (host pcbnew 5.1.6)
+(kicad_pcb (version 20171130) (host pcbnew 5.1.8)
   (general
     (thickness 1.6)
-    (drawings 9)
+    (drawings 22)
     (tracks 304)
     (zones 0)
-    (modules 113)
+    (modules 109)
     (nets 41)
   )
@@
     )
   )
+  (gr_text "GND\nDATA\n5V" (at 134.3 128.4 90) (layer F.SilkS)
+    (effects (font (size 0.6 0.6) (thickness 0.15)))
+  )
+  (gr_text "WS2812 1" (at 146.4 126.8 90) (layer F.SilkS)
+    (effects (font (size 0.7 0.7) (thickness 0.15)))
+  )
+  (gr_text "WS2812 0" (at 159.1 126.8 90) (layer F.SilkS)
+    (effects (font (size 0.7 0.7) (thickness 0.15)))
+  )
+  (gr_text "B\nR\nG\n12V" (at 163.3 128.4 90) (layer F.SilkS)
+    (effects (font (size 0.6 0.6) (thickness 0.15)))
+  )
+  (gr_text "12V PWM 1" (at 178.2 126.6 90) (layer F.SilkS)
+    (effects (font (size 0.7 0.7) (thickness 0.15)))
+  )
+  (gr_text "12V PWM 0" (at 193.5 126.7 90) (layer F.SilkS)
+    (effects (font (size 0.7 0.7) (thickness 0.15)))
+  )
+  (gr_text "LED Power" (at 190.9 103.2 90) (layer F.SilkS)
+    (effects (font (size 0.7 0.7) (thickness 0.15)))
+  )
+  (gr_text "12V\nGND\nGND\nGND" (at 176.1 101.4 90) (layer F.SilkS)
+    (effects (font (size 0.6 0.6) (thickness 0.15)))
+  )
+  (gr_text "5V\nD-\nD+\nGND" (at 138.6 101.5 90) (layer F.SilkS)
+    (effects (font (size 0.6 0.6) (thickness 0.15)))
+  )
+  (gr_text USB (at 153.4 102.9 90) (layer F.SilkS)
+    (effects (font (size 0.75 0.75) (thickness 0.15)))
+  )
+  (gr_text http://kevincuzner.com (at 192.5 112.5 90) (layer F.SilkS)
+    (effects (font (size 1 1) (thickness 0.15)))
+  )
+  (gr_text "Rev A" (at 137.1 108.2 270) (layer F.SilkS)
+    (effects (font (size 1 1) (thickness 0.15)))
+  )
+  (gr_text "USB LED Controller" (at 138.6 113.4 270) (layer F.SilkS)
+    (effects (font (size 1 1) (thickness 0.15)))
+  )
   (dimension 4.14 (width 0.15) (layer Dwgs.User)
